File: prelimHolocube/pcb/v3/test_single-board/test_single-board.kicad_sch (KiCad schematic)
At the start: 0 parts

Commit message: finish kicad for single board
Parts:
- added C1, C3: 4.7uF, Capacitor_THT:CP_Radial_D4.0mm_P2.00mm, symbol Device:C_US
- added C2: 1uF ceramic, Capacitor_THT:C_Disc_D6.0mm_W2.5mm_P5.00mm, symbol Device:C
- added R1: 1M, Resistor_THT:R_Axial_DIN0207_L6.3mm_D2.5mm_P7.62mm_Horizontal, symbol Device:R_US
- added U1: ~, transparent_oled_display:surenoo-1.12in-128x128, symbol transparent_oled_display:surenoo-1.12in-128x128
- added U10: ~, Connector_PinHeader_2.54mm:PinHeader_1x02_P2.54mm_Vertical, symbol Power_Supply:DC_2-Terminals
- added U9: ~, esp32:devkitv1-30pin, symbol esp32:devkitv1-30pin
Connections:
- new net: R1.1, U1.7 (IREF)
- new net: C1.1, U1.10 (VCOMH)
- new net +13.5V: C3.1, U1.11 (VPP), U10.1 (VCC)
- new net +3.3V: C2.2, U1.8 (VDD), U9.16 (3V3)
- new net A0: U1.4 (A0), U9.21 (RX2)
- new net CS: U1.6 (CS), U9.22 (TX2)
- new net GND: C1.2, C2.1, C3.2, R1.2, U1.1 (VSS), U1.12 (VSS), U1.9 (VSS), U10.2 (GND), U9.17 (GND), U9.2 (GND)
- new net RES: U1.5 (RES), U9.20 (D4)
- new net SCL: U1.3 (SCL), U9.24 (D18)
- new net SI: U1.2 (SI), U9.30 (D23)
