File: prelimHolocube/pcb/v1.0/test_single-board/test_single-board.kicad_pcb (KiCad board)
At the start: 2 copper layers, 56.5 x 53.9 mm, 7 parts

Commit message: Finish multiboard pcb
Other:
- board text added: "Holocube v1.0 Testing Phase: Single-Board"
- board text removed: "Holocube v3 Testing Phase: Single-Board"
Changed lines of the file:
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@@
 		)
 	)
-	(gr_text "Holocube v3\nTesting Phase: Single-Board"
+	(gr_text "Holocube v1.0\nTesting Phase: Single-Board"
 		(at 167.915 68.726 0)
 		(layer "F.SilkS")
