File: prelimHolocube/pcb/v1.0/main/holocube.kicad_sch (KiCad schematic)
At the start: 51 parts, among them J1 USB_C_Receptacle_USB2.0_14P, U11 KY-040

Commit message: Place v1.0 footprints on pcb and link 3d models
Parts:
- removed C25: 10nF 100V, Capacitor_SMD:C_0805_2012Metric, symbol Device:C
- removed J1: USB_C_Receptacle_USB2.0_14P, Connector_USB:USB_C_Receptacle_GCT_USB4105-xx-A_16P_TopMnt_Horizontal, symbol Connector:USB_C_Receptacle_USB2.0_14P
- removed R10: 1M, symbol Device:R_US
- added C26: 10nF 100V, Capacitor_SMD:C_0603_1608Metric, symbol Device:C
- added J2: USB4105-GF-A, usbc_connector:usbc_connector, symbol usbc_connector:USB4105-GF-A
- added R14: 1M, Resistor_SMD:R_0805_2012Metric, symbol Device:R_US
- C1, C11, C12, C14, C16, C17, C18, C20, C22, C23, C24, C3, C5, C6, C8, C9: footprint Capacitor_THT:CP_Radial_D4.0mm_P2.00mm -> Capacitor_SMD:CP_Elec_4x5.4
- C10, C13, C15, C19, C2, C21, C4, C7: footprint Capacitor_THT:CP_Radial_D5.0mm_P2.50mm -> Capacitor_SMD:C_0805_2012Metric
- D1: footprint (none) -> LED_SMD:LED_0603_1608Metric
- R1, R2, R3, R4, R5, R6, R7, R8: footprint Resistor_THT:R_Axial_DIN0207_L6.3mm_D2.5mm_P7.62mm_Horizontal -> Resistor_SMD:R_0805_2012Metric
- R11, R12, R9: footprint (none) -> Resistor_SMD:R_0805_2012Metric
- R13: value 330 -> 68; footprint (none) -> Resistor_SMD:R_0805_2012Metric
- U1, U2, U3, U4, U5, U6, U7, U8: footprint transparent_oled_display:surenoo-1.12in-128x128 -> Vertical_FPC-Connector_12P:AMPHENOL_F31W-1A7H1-11012
- U10: footprint (none) -> boost_converter:Dorhea_MT3608_Adjustable
- U11: footprint KY-040:KY-040-PORT -> KY-040:KY-040
Connections:
- net +5V: now also J2.A4_B9 (VBUS), J2.B4_A9 (VBUS)
- net GND: now also U1.SH1 (Shield), U2.SH1 (Shield), U3.SH1 (Shield), U4.SH1 (Shield), U5.SH1 (Shield), U6.SH1 (Shield), U7.SH1 (Shield), U8.SH1 (Shield), C26.2, J2.A1_B12 (GND), J2.B1_A12 (GND), R14.2
- net LED: now also U9.20 (D4)
- net at R11.1: now also J2.A5 (CC1)
- net at R12.1: now also J2.B5 (CC2)
- new net SHELL_GND: C26.1, J2.SH1 (SHELL_GND), J2.SH2 (SHELL_GND), J2.SH3 (SHELL_GND), J2.SH4 (SHELL_GND), R14.1
- no-connect marks 4 -> 6
Other:
- moved on the sheet: R11, R12, U10

Commit message: order multiboard and update full board
Parts:
- removed R9: 10k, Resistor_SMD:R_0805_2012Metric, symbol Device:R_US
- removed U10: ~, boost_converter:Dorhea_MT3608_Adjustable, symbol boost_converter:Dorhea_MT3608_Adjustable
- added U10: ~, boost_converter:HiLetgo_XL6009_Adjustable, symbol boost_converter:HiLetgo_XL6009_Adjustable
Connections:
- net +13.5V: now also U10.1 (VOUT+)
- net +3.3V: now also U11.VCC
- net GND: now also U10.2 (VOUT-), U10.4 (VIN-)
- net KY_SW: now also U9.29 (D22)
- net VBUS: now reaches U9.1 (VIN)
- net VBUS: now also J2.A4_B9 (VBUS), J2.B4_A9 (VBUS), U10.3 (VIN+)
- removed net +5V: J2.A4_B9 (VBUS), J2.B4_A9 (VBUS), U11.VCC
- no-connect marks 6 -> 15
Other:
- note added: "USB-C used for MCU logic power and serial uploading."
- note removed: "MicroUSB used for MCU logic power and serial uploading."
