File: prelimHolocube/pcb/v1.0/main/holocube.kicad_pcb (KiCad board)
At the start: 2 copper layers, 54.5 x 54.5 mm, 54 parts, among them J2 USB4105-GF-A, U11 KY-040

Commit message: Update holocube.kicad_pcb
Parts:
- moved R1 13.7 mm to (162.0, 79.8)
- moved R2 13.7 mm to (162.0, 84.8)
- moved R4 13.7 mm to (161.9, 94.8)
- moved R5 13.7 mm to (161.9, 99.5)
- moved R6 13.7 mm to (161.9, 104.5)
- moved R7 13.7 mm to (161.9, 109.4)
- moved R8 13.7 mm to (161.9, 114.4)
- moved R3 13.7 mm to (162.0, 89.7)
- moved U3 2.03 mm to (169.9, 90.1)
- moved U4 2.03 mm to (169.9, 95.1)
- moved U5 2.03 mm to (169.9, 100.0)
- moved U6 2.03 mm to (169.9, 105.0)
- moved U7 2.03 mm to (169.8, 109.9)
- moved U8 2.03 mm to (169.8, 114.9)
- moved U2 2.02 mm to (169.9, 85.2)
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Routing:
- net GND: track 145.6 -> 21.7 mm, vias 34 -> 5
- net CS2: track 0.00 -> 42.4 mm
- net CS1: track 40.6 -> 0.00 mm, vias 2 -> 0
- net Net-(U2-VCOMH): track 0.00 -> 14.1 mm
- net Net-(U1-VCOMH): track 13.1 -> 0.00 mm
- net RES: track 56.6 -> 46.6 mm
- net Net-(U1-IREF): track 9.70 -> 0.00 mm
- net Net-(U2-IREF): track 0.00 -> 8.91 mm
- net SCL: track 60.3 -> 51.8 mm, vias 8 -> 9
- net SI: track 60.1 -> 52.2 mm
- net A0: track 57.4 -> 50.8 mm, vias 8 -> 9
- net +13.5V: track 129.2 -> 132.4 mm, vias 4 -> 9

Commit message: fully route main v1.0 + gerbers
Routing:
- net GND: track 21.7 -> 323.8 mm, vias 5 -> 84
- net +13.5V: track 132.4 -> 313.5 mm, vias 9 -> 22
- net +3.3V: track 77.7 -> 185.9 mm
- net CS3: track 0.00 -> 42.6 mm, vias 0 -> 2
- net CS5: track 0.00 -> 42.3 mm, vias 0 -> 2
- net CS4: track 0.00 -> 42.1 mm, vias 0 -> 2
- net CS6: track 0.00 -> 41.7 mm, vias 0 -> 2
- net CS1: track 0.00 -> 41.7 mm, vias 0 -> 2
- net CS7: track 0.00 -> 40.0 mm, vias 0 -> 5
- net CS8: track 0.00 -> 38.7 mm, vias 0 -> 6
- net LED: track 0.00 -> 34.4 mm, vias 0 -> 2
- net KY_CLK: track 0.00 -> 32.2 mm, vias 0 -> 1
- net KY_DT: track 0.00 -> 29.9 mm, vias 0 -> 1
- net KY_SW: track 0.00 -> 27.3 mm, vias 0 -> 3
- net SCL: track 51.8 -> 78.1 mm, vias 9 -> 10
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Other:
- board text added: "Last updated: 09/27/26 Made with love :)"
- board text removed: "Last updated: 09/22/26 Made with love :)"
